File: environment-sensor-sip-baseboard.kicad_pcb (KiCad board)
At the start: 4 copper layers, 50 x 26.5 mm, 59 parts, among them J1 USB-C_GCT_USB4105-GF-A, J2 JST_SH_1x4_SM04B-SRSS-TB-LF-SN, J3 JST_SH_1x4_SM04B-SRSS-TB-LF-SN, U1 Antmicro_GEM3, U5 SHT45, U6 BME280

Commit message: [#62396] Update components
Parts:
- U1: value Antmicro_GEM3 -> Myra-231F1F08; footprint antmicro-footprints:LGA-64_11.4x11.4mm_GEM3-footprint -> antmicro-footprints:LGA-64_11.4x11.4mm_Myra
Connections:
- U1 pad B1: GND -> unconnected-(U1-PadB1)
- U1 pad C1: GND -> unconnected-(U1-PadC1)

Commit message: [#62396] Fix ERC and DRC
Connections:
- U1 pad B1: unconnected-(U1-PadB1) -> GND
- U1 pad C1: unconnected-(U1-PadC1) -> GND

Commit message: [#62396] Update SiP
Other:
- board text added: "PCB SHA c359ffe9"
- board text removed: "PCB SHA ########"
